File: games/switched-tag/logic-circuit/kicad-circuit/switched-tag-circuit-kicad/switched-tag-abs-zero-detector.kicad_sch (KiCad schematic)
At the start: 19 parts

Commit message: Saving progress.
Parts:
- U6, U7, U8, U9: Spice_Lib_File /home/pab/Inventions/analog-circuit-game-console/ms-circuit-video-games/spice-models/lmx58_lm2904.lib -> /home/pab/Inventions/analog-circuit-game-console/ms-circuit-video-games/spice-models/ad8031.mod; Spice_Model LMX58_LM2904 -> AD8031
Changed lines of the file:
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@@
       (effects (font (size 1.27 1.27)) (justify left) hide)
     )
-    (property "Spice_Model" "LMX58_LM2904" (id 6) (at 180.34 99.06 0)
-      (effects (font (size 1.27 1.27)) hide)
-    )
-    (property "Spice_Lib_File" "/home/pab/Inventions/analog-circuit-game-console/ms-circuit-video-games/spice-models/lmx58_lm2904.lib" (id 7) (at 180.34 99.06 0)
+    (property "Spice_Model" "AD8031" (id 6) (at 180.34 99.06 0)
+      (effects (font (size 1.27 1.27)) hide)
+    )
+    (property "Spice_Lib_File" "/home/pab/Inventions/analog-circuit-game-console/ms-circuit-video-games/spice-models/ad8031.mod" (id 7) (at 180.34 99.06 0)
       (effects (font (size 1.27 1.27)) hide)
     )
@@
       (effects (font (size 1.27 1.27)) (justify left) hide)
     )
-    (property "Spice_Model" "LMX58_LM2904" (id 6) (at 114.3 101.6 0)
-      (effects (font (size 1.27 1.27)) hide)
-    )
-    (property "Spice_Lib_File" "/home/pab/Inventions/analog-circuit-game-console/ms-circuit-video-games/spice-models/lmx58_lm2904.lib" (id 7) (at 114.3 101.6 0)
+    (property "Spice_Model" "AD8031" (id 6) (at 114.3 101.6 0)
+      (effects (font (size 1.27 1.27)) hide)
+    )
+    (property "Spice_Lib_File" "/home/pab/Inventions/analog-circuit-game-console/ms-circuit-video-games/spice-models/ad8031.mod" (id 7) (at 114.3 101.6 0)
       (effects (font (size 1.27 1.27)) hide)
     )
@@
       (effects (font (size 1.27 1.27)) (justify left) hide)
     )
-    (property "Spice_Model" "LMX58_LM2904" (id 6) (at 62.23 100.33 0)
-      (effects (font (size 1.27 1.27)) hide)
-    )
-    (property "Spice_Lib_File" "/home/pab/Inventions/analog-circuit-game-console/ms-circuit-video-games/spice-models/lmx58_lm2904.lib" (id 7) (at 62.23 100.33 0)
+    (property "Spice_Model" "AD8031" (id 6) (at 62.23 100.33 0)
+      (effects (font (size 1.27 1.27)) hide)
+    )
+    (property "Spice_Lib_File" "/home/pab/Inventions/analog-circuit-game-console/ms-circuit-video-games/spice-models/ad8031.mod" (id 7) (at 62.23 100.33 0)
       (effects (font (size 1.27 1.27)) hide)
     )
@@
       (effects (font (size 1.27 1.27)) (justify left) hide)
     )
-    (property "Spice_Model" "LMX58_LM2904" (id 6) (at 231.14 111.76 0)
-      (effects (font (size 1.27 1.27)) hide)
-    )
-    (property "Spice_Lib_File" "/home/pab/Inventions/analog-circuit-game-console/ms-circuit-video-games/spice-models/lmx58_lm2904.lib" (id 7) (at 231.14 111.76 0)
-      (effects (font (size 1.27 1.27)) hide)
-    )
+    (property "Spice_Model" "AD8031" (id 6) (at 231.14 111.76 0)
+      (effects (font (size 1.27 1.27)) hide)
+    )
+    (property "Spice_Lib_File" "/home/pab/Inventions/analog-circuit-game-console/ms-circuit-video-games/spice-models/ad8031.mod" (id 7) (at 231.14 111.76 0)
+      (effects (font (size 1.27 1.27)) hide)
+    )
