File: games/switched-tag/logic-circuit/kicad-circuit/switched-tag-circuit-kicad/switched-tag-pendelum-model.kicad_sch (KiCad schematic)
At the start: 7 parts

Commit message: Added some prep work for console hardware.
Parts:
- U17, U18, U19: Spice_Lib_File /home/pab/Inventions/analog-circuit-game-console/ms-circuit-video-games/spice-models/ada4692.mod -> /home/pab/Inventions/analog-circuit-game-console/ms-circuit-video-games/spice-models/lmx58_lm2904.lib; Spice_Model ADA4692 -> LMX58_LM2904
Changed lines of the file:
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@@
       (effects (font (size 1.27 1.27)) (justify left) hide)
     )
-    (property "Spice_Model" "ADA4692" (id 6) (at 163.83 58.42 0)
+    (property "Spice_Model" "LMX58_LM2904" (id 6) (at 163.83 58.42 0)
       (effects (font (size 1.27 1.27)) hide)
     )
-    (property "Spice_Lib_File" "/home/pab/Inventions/analog-circuit-game-console/ms-circuit-video-games/spice-models/ada4692.mod" (id 7) (at 163.83 58.42 0)
+    (property "Spice_Lib_File" "/home/pab/Inventions/analog-circuit-game-console/ms-circuit-video-games/spice-models/lmx58_lm2904.lib" (id 7) (at 163.83 58.42 0)
       (effects (font (size 1.27 1.27)) hide)
     )
@@
       (effects (font (size 1.27 1.27)) (justify left) hide)
     )
-    (property "Spice_Model" "ADA4692" (id 6) (at 78.74 85.09 0)
+    (property "Spice_Model" "LMX58_LM2904" (id 6) (at 78.74 85.09 0)
       (effects (font (size 1.27 1.27)) hide)
     )
-    (property "Spice_Lib_File" "/home/pab/Inventions/analog-circuit-game-console/ms-circuit-video-games/spice-models/ada4692.mod" (id 7) (at 78.74 85.09 0)
+    (property "Spice_Lib_File" "/home/pab/Inventions/analog-circuit-game-console/ms-circuit-video-games/spice-models/lmx58_lm2904.lib" (id 7) (at 78.74 85.09 0)
       (effects (font (size 1.27 1.27)) hide)
     )
@@
       (effects (font (size 1.27 1.27)) (justify left) hide)
     )
-    (property "Spice_Model" "ADA4692" (id 6) (at 119.38 87.63 0)
+    (property "Spice_Model" "LMX58_LM2904" (id 6) (at 119.38 87.63 0)
       (effects (font (size 1.27 1.27)) hide)
     )
-    (property "Spice_Lib_File" "/home/pab/Inventions/analog-circuit-game-console/ms-circuit-video-games/spice-models/ada4692.mod" (id 7) (at 119.38 87.63 0)
+    (property "Spice_Lib_File" "/home/pab/Inventions/analog-circuit-game-console/ms-circuit-video-games/spice-models/lmx58_lm2904.lib" (id 7) (at 119.38 87.63 0)
       (effects (font (size 1.27 1.27)) hide)
     )

Commit message: Saving progress.
Parts:
- U17, U18, U19: Spice_Lib_File /home/pab/Inventions/analog-circuit-game-console/ms-circuit-video-games/spice-models/lmx58_lm2904.lib -> /home/pab/Inventions/analog-circuit-game-console/ms-circuit-video-games/spice-models/ad8031.mod; Spice_Model LMX58_LM2904 -> AD8031
Changed lines of the file:
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@@
       (effects (font (size 1.27 1.27)) (justify left) hide)
     )
-    (property "Spice_Model" "LMX58_LM2904" (id 6) (at 163.83 58.42 0)
+    (property "Spice_Model" "AD8031" (id 6) (at 163.83 58.42 0)
       (effects (font (size 1.27 1.27)) hide)
     )
-    (property "Spice_Lib_File" "/home/pab/Inventions/analog-circuit-game-console/ms-circuit-video-games/spice-models/lmx58_lm2904.lib" (id 7) (at 163.83 58.42 0)
+    (property "Spice_Lib_File" "/home/pab/Inventions/analog-circuit-game-console/ms-circuit-video-games/spice-models/ad8031.mod" (id 7) (at 163.83 58.42 0)
       (effects (font (size 1.27 1.27)) hide)
     )
@@
       (effects (font (size 1.27 1.27)) (justify left) hide)
     )
-    (property "Spice_Model" "LMX58_LM2904" (id 6) (at 78.74 85.09 0)
+    (property "Spice_Model" "AD8031" (id 6) (at 78.74 85.09 0)
       (effects (font (size 1.27 1.27)) hide)
     )
-    (property "Spice_Lib_File" "/home/pab/Inventions/analog-circuit-game-console/ms-circuit-video-games/spice-models/lmx58_lm2904.lib" (id 7) (at 78.74 85.09 0)
+    (property "Spice_Lib_File" "/home/pab/Inventions/analog-circuit-game-console/ms-circuit-video-games/spice-models/ad8031.mod" (id 7) (at 78.74 85.09 0)
       (effects (font (size 1.27 1.27)) hide)
     )
@@
       (effects (font (size 1.27 1.27)) (justify left) hide)
     )
-    (property "Spice_Model" "LMX58_LM2904" (id 6) (at 119.38 87.63 0)
+    (property "Spice_Model" "AD8031" (id 6) (at 119.38 87.63 0)
       (effects (font (size 1.27 1.27)) hide)
     )
-    (property "Spice_Lib_File" "/home/pab/Inventions/analog-circuit-game-console/ms-circuit-video-games/spice-models/lmx58_lm2904.lib" (id 7) (at 119.38 87.63 0)
+    (property "Spice_Lib_File" "/home/pab/Inventions/analog-circuit-game-console/ms-circuit-video-games/spice-models/ad8031.mod" (id 7) (at 119.38 87.63 0)
       (effects (font (size 1.27 1.27)) hide)
     )
