File: games/switched-tag/logic-circuit/kicad-circuit/switched-tag-circuit-kicad/switched-tag-sample-and-hold.kicad_sch (KiCad schematic)
At the start: 4 parts, among them Q1 RUL035N02

Commit message: Added some prep work for console hardware.
Parts:
- Q1: value RUL035N02 -> (none); Spice_Lib_File /home/pab/Inventions/analog-circuit-game-console/ms-circuit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 -> ../../../../../spice-models/rul035n02.lib
- U13, U14: Spice_Lib_File /home/pab/Inventions/analog-circuit-game-console/ms-circuit-video-games/spice-models/ada4692.mod -> /home/pab/Inventions/analog-circuit-game-console/ms-circuit-video-games/spice-models/lmx58_lm2904.lib; Spice_Model ADA4692 -> LMX58_LM2904
Changed lines of the file:
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@@
       (effects (font (size 1.27 1.27)) (justify left) hide)
     )
-    (property "Spice_Model" "ADA4692" (id 6) (at 193.04 92.71 0)
+    (property "Spice_Model" "LMX58_LM2904" (id 6) (at 193.04 92.71 0)
       (effects (font (size 1.27 1.27)) hide)
     )
-    (property "Spice_Lib_File" "/home/pab/Inventions/analog-circuit-game-console/ms-circuit-video-games/spice-models/ada4692.mod" (id 7) (at 193.04 92.71 0)
+    (property "Spice_Lib_File" "/home/pab/Inventions/analog-circuit-game-console/ms-circuit-video-games/spice-models/lmx58_lm2904.lib" (id 7) (at 193.04 92.71 0)
       (effects (font (size 1.27 1.27)) hide)
     )
@@
       (effects (font (size 1.27 1.27)) (justify left) hide)
     )
-    (property "Spice_Model" "ADA4692" (id 6) (at 118.11 93.98 0)
+    (property "Spice_Model" "LMX58_LM2904" (id 6) (at 118.11 93.98 0)
       (effects (font (size 1.27 1.27)) hide)
     )
-    (property "Spice_Lib_File" "/home/pab/Inventions/analog-circuit-game-console/ms-circuit-video-games/spice-models/ada4692.mod" (id 7) (at 118.11 93.98 0)
+    (property "Spice_Lib_File" "/home/pab/Inventions/analog-circuit-game-console/ms-circuit-video-games/spice-models/lmx58_lm2904.lib" (id 7) (at 118.11 93.98 0)
       (effects (font (size 1.27 1.27)) hide)
     )
@@
       (effects (font (size 1.27 1.27)) (justify left))
     )
-    (property "Value" "RUL035N02" (id 1) (at 153.67 106.6799 0)
+    (property "Value" "" (id 1) (at 153.67 106.6799 0)
       (effects (font (size 1.27 1.27)) (justify left))
     )
@@
       (effects (font (size 1.27 1.27)) hide)
     )
-    (property "Spice_Lib_File" "/home/pab/Inventions/analog-circuit-game-console/ms-circuit-video-games/spice-models/rul035n02.lib" (id 7) (at 147.32 105.41 0)
+    (property "Spice_Lib_File" "../../../../../spice-models/rul035n02.lib" (id 7) (at 147.32 105.41 0)
       (effects (font (size 1.27 1.27)) hide)
     )

Commit message: Saving progress.
Parts:
- U13, U14: Spice_Lib_File /home/pab/Inventions/analog-circuit-game-console/ms-circuit-video-games/spice-models/lmx58_lm2904.lib -> /home/pab/Inventions/analog-circuit-game-console/ms-circuit-video-games/spice-models/ad8031.mod; Spice_Model LMX58_LM2904 -> AD8031
Changed lines of the file:
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@@
       (effects (font (size 1.27 1.27)) (justify left) hide)
     )
-    (property "Spice_Model" "LMX58_LM2904" (id 6) (at 193.04 92.71 0)
+    (property "Spice_Model" "AD8031" (id 6) (at 193.04 92.71 0)
       (effects (font (size 1.27 1.27)) hide)
     )
-    (property "Spice_Lib_File" "/home/pab/Inventions/analog-circuit-game-console/ms-circuit-video-games/spice-models/lmx58_lm2904.lib" (id 7) (at 193.04 92.71 0)
+    (property "Spice_Lib_File" "/home/pab/Inventions/analog-circuit-game-console/ms-circuit-video-games/spice-models/ad8031.mod" (id 7) (at 193.04 92.71 0)
       (effects (font (size 1.27 1.27)) hide)
     )
@@
       (effects (font (size 1.27 1.27)) (justify left) hide)
     )
-    (property "Spice_Model" "LMX58_LM2904" (id 6) (at 118.11 93.98 0)
+    (property "Spice_Model" "AD8031" (id 6) (at 118.11 93.98 0)
       (effects (font (size 1.27 1.27)) hide)
     )
-    (property "Spice_Lib_File" "/home/pab/Inventions/analog-circuit-game-console/ms-circuit-video-games/spice-models/lmx58_lm2904.lib" (id 7) (at 118.11 93.98 0)
+    (property "Spice_Lib_File" "/home/pab/Inventions/analog-circuit-game-console/ms-circuit-video-games/spice-models/ad8031.mod" (id 7) (at 118.11 93.98 0)
       (effects (font (size 1.27 1.27)) hide)
     )
