File: games/switched-tag/analog-module/pcb/switched-tag-circuit-kicad/switched-tag-collision-detection.kicad_sch (KiCad schematic)
At the start: 40 parts, among them U14 TLV9154IDR, U15 TLV9154IDR

Commit message: Saving pcb placement.
Parts:
- U14, U15: footprint SOIC_9154IDR_TEX -> switched-tag-footprint-lib:SOIC_9154IDR_TEX
Connections:
- net GND1: now also U15.10 (IN3+), U15.12 (IN4+); no longer U15.3 (IN1+), U15.5 (IN2+)
- net U3_V-: now also U14.13 (IN4-); no longer U14.9 (IN3-)
- net U3_Vout: now also U14.14 (OUT4), U15.13 (IN4-); no longer U14.8 (OUT3), U15.2 (IN1-)
- net U4_V-: now also U14.9 (IN3-); no longer U14.13 (IN4-)
- net U4_Vout: now also U14.8 (OUT3), U15.9 (IN3-); no longer U14.14 (OUT4), U15.6 (IN2-)
- net U5_Vout: now also U15.14 (OUT4); no longer U15.1 (OUT1)
- net U6_Vout: now also U15.8 (OUT3); no longer U15.7 (OUT2)
- net U7_V+: now also U15.3 (IN1+); no longer U15.10 (IN3+)
- net U7_V-: now also U15.2 (IN1-); no longer U15.9 (IN3-)
- net U7_Vout: now also U15.1 (OUT1), U15.6 (IN2-); no longer U15.13 (IN4-), U15.8 (OUT3)
- net U8_V+: now also U15.5 (IN2+); no longer U15.12 (IN4+)
- net U8_Vout: now also U15.7 (OUT2); no longer U15.14 (OUT4)
Changed lines of the file:
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@@
     (effects (font (size 1.27 1.27)) (justify left bottom))
   )
-  (label "U7_V-" (at 270.51 35.56 180) (fields_autoplaced)
+  (label "U7_V-" (at 270.51 25.4 180) (fields_autoplaced)
     (effects (font (size 1.27 1.27)) (justify right bottom))
   )
@@
     (effects (font (size 1.27 1.27)) (justify left bottom))
   )
-  (label "U8_Vout" (at 320.04 30.48 0) (fields_autoplaced)
+  (label "U8_Vout" (at 320.04 25.4 0) (fields_autoplaced)
     (effects (font (size 1.27 1.27)) (justify left bottom))
   )
@@
     (effects (font (size 1.27 1.27)) (justify left bottom))
   )
-  (label "U6_V-" (at 270.51 30.48 180) (fields_autoplaced)
+  (label "U6_V-" (at 270.51 35.56 180) (fields_autoplaced)
     (effects (font (size 1.27 1.27)) (justify right bottom))
   )
@@
     (effects (font (size 1.27 1.27)) (justify right bottom))
   )
-  (label "U3_V-" (at 196.85 35.56 180) (fields_autoplaced)
-    (effects (font (size 1.27 1.27)) (justify right bottom))
-  )
-  (label "U3_V+" (at 196.85 38.1 180) (fields_autoplaced)
+  (label "U3_V-" (at 196.85 40.64 180) (fields_autoplaced)
+    (effects (font (size 1.27 1.27)) (justify right bottom))
+  )
+  (label "U3_V+" (at 196.85 43.18 180) (fields_autoplaced)
     (effects (font (size 1.27 1.27)) (justify right bottom))
   )
@@
     (effects (font (size 1.27 1.27)) (justify left bottom))
   )
-  (label "U8_V+" (at 270.51 43.18 180) (fields_autoplaced)
-    (effects (font (size 1.27 1.27)) (justify right bottom))
-  )
-  (label "U3_Vout" (at 246.38 27.94 0) (fields_autoplaced)
-    (effects (font (size 1.27 1.27)) (justify left bottom))
-  )
-  (label "U7_V+" (at 270.51 38.1 180) (fields_autoplaced)
-    (effects (font (size 1.27 1.27)) (justify right bottom))
-  )
-  (label "U5_V+" (at 270.51 27.94 180) (fields_autoplaced)
+  (label "U8_V+" (at 270.51 33.02 180) (fields_autoplaced)
+    (effects (font (size 1.27 1.27)) (justify right bottom))
+  )
+  (label "U3_Vout" (at 246.38 30.48 0) (fields_autoplaced)
+    (effects (font (size 1.27 1.27)) (justify left bottom))
+  )
+  (label "U7_V+" (at 270.51 27.94 180) (fields_autoplaced)
+    (effects (font (size 1.27 1.27)) (justify right bottom))
+  )
+  (label "U5_V+" (at 270.51 43.18 180) (fields_autoplaced)
     (effects (font (size 1.27 1.27)) (justify right bottom))
   )
@@
     (effects (font (size 1.27 1.27)) (justify left bottom))
   )
-  (label "U5_Vout" (at 320.04 22.86 0) (fields_autoplaced)
+  (label "U5_Vout" (at 320.04 30.48 0) (fields_autoplaced)
     (effects (font (size 1.27 1.27)) (justify left bottom))
   )
@@
     (effects (font (size 1.27 1.27)) (justify left bottom))
   )
-  (label "U6_V+" (at 270.51 33.02 180) (fields_autoplaced)
+  (label "U6_V+" (at 270.51 38.1 180) (fields_autoplaced)
     (effects (font (size 1.27 1.27)) (justify right bottom))
   )
@@
     (effects (font (size 1.27 1.27)) (justify right bottom))
   )
-  (label "U6_Vout" (at 320.04 25.4 0) (fields_autoplaced)
-    (effects (font (size 1.27 1.27)) (justify left bottom))
-  )
-  (label "U5_V-" (at 270.51 25.4 180) (fields_autoplaced)
+  (label "U6_Vout" (at 320.04 27.94 0) (fields_autoplaced)
+    (effects (font (size 1.27 1.27)) (justify left bottom))
+  )
+  (label "U5_V-" (at 270.51 40.64 180) (fields_autoplaced)
     (effects (font (size 1.27 1.27)) (justify right bottom))
   )
@@
     (effects (font (size 1.27 1.27)) (justify left bottom))
   )
-  (label "U4_Vout" (at 246.38 30.48 0) (fields_autoplaced)
+  (label "U4_Vout" (at 246.38 27.94 0) (fields_autoplaced)
     (effects (font (size 1.27 1.27)) (justify left bottom))
   )
@@
     (effects (font (size 1.27 1.27)) (justify right bottom))
   )
-  (label "U4_V+" (at 196.85 43.18 180) (fields_autoplaced)
+  (label "U4_V+" (at 196.85 38.1 180) (fields_autoplaced)
     (effects (font (size 1.27 1.27)) (justify right bottom))
   )
@@
     (effects (font (size 1.27 1.27)) (justify right bottom))
   )
-  (label "U8_V-" (at 270.51 40.64 180) (fields_autoplaced)
-    (effects (font (size 1.27 1.27)) (justify right bottom))
-  )
-  (label "U4_V-" (at 196.85 40.64 180) (fields_autoplaced)
+  (label "U8_V-" (at 270.51 30.48 180) (fields_autoplaced)
+    (effects (font (size 1.27 1.27)) (justify right bottom))
+  )
+  (label "U4_V-" (at 196.85 35.56 180) (fields_autoplaced)
     (effects (font (size 1.27 1.27)) (justify right bottom))
   )
@@
     (effects (font (size 1.27 1.27)) (justify left bottom))
   )
-  (label "U7_Vout" (at 320.04 27.94 0) (fields_autoplaced)
+  (label "U7_Vout" (at 320.04 22.86 0) (fields_autoplaced)
     (effects (font (size 1.27 1.27)) (justify left bottom))
   )
@@
       (effects (font (size 1.524 1.524)))
     )
-    (property "Footprint" "SOIC_9154IDR_TEX" (at 201.93 25.4 0)
+    (property "Footprint" "switched-tag-footprint-lib:SOIC_9154IDR_TEX" (at 201.93 25.4 0)
       (effects (font (size 1.27 1.27) italic) hide)
     )
@@
       (effects (font (size 1.524 1.524)))
     )
-    (property "Footprint" "SOIC_9154IDR_TEX" (at 274.32 25.4 0)
+    (property "Footprint" "switched-tag-footprint-lib:SOIC_9154IDR_TEX" (at 274.32 25.4 0)
       (effects (font (size 1.27 1.27) italic) hide)
     )

Commit message: Changed component size from 0603 to 0805 for easier hand soldering.
Parts:
- D? (x5): footprint Diode_SMD:D_0603_1608Metric -> Diode_SMD:D_0805_2012Metric
- R? (x25): footprint Resistor_SMD:R_0603_1608Metric -> Resistor_SMD:R_0805_2012Metric
Changed lines of the file:
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@@
       (effects (font (size 1.27 1.27)))
     )
-    (property "Footprint" "Resistor_SMD:R_0603_1608Metric" (at 214.63 110.998 90)
+    (property "Footprint" "Resistor_SMD:R_0805_2012Metric" (at 214.63 110.998 90)
       (effects (font (size 1.27 1.27)) hide)
     )
@@
       (effects (font (size 1.27 1.27)))
     )
-    (property "Footprint" "Resistor_SMD:R_0603_1608Metric" (at 119.38 82.042 90)
+    (property "Footprint" "Resistor_SMD:R_0805_2012Metric" (at 119.38 82.042 90)
       (effects (font (size 1.27 1.27)) hide)
     )
@@
       (effects (font (size 1.27 1.27)))
     )
-    (property "Footprint" "Resistor_SMD:R_0603_1608Metric" (at 102.87 174.498 90)
+    (property "Footprint" "Resistor_SMD:R_0805_2012Metric" (at 102.87 174.498 90)
       (effects (font (size 1.27 1.27)) hide)
     )
@@
       (effects (font (size 1.27 1.27)))
     )
-    (property "Footprint" "Resistor_SMD:R_0603_1608Metric" (at 190.5 95.758 90)
+    (property "Footprint" "Resistor_SMD:R_0805_2012Metric" (at 190.5 95.758 90)
       (effects (font (size 1.27 1.27)) hide)
     )
@@
       (effects (font (size 1.27 1.27)))
     )
-    (property "Footprint" "Resistor_SMD:R_0603_1608Metric" (at 46.99 72.898 90)
+    (property "Footprint" "Resistor_SMD:R_0805_2012Metric" (at 46.99 72.898 90)
       (effects (font (size 1.27 1.27)) hide)
     )
@@
       (effects (font (size 1.27 1.27)))
     )
-    (property "Footprint" "Resistor_SMD:R_0603_1608Metric" (at 46.99 126.238 90)
+    (property "Footprint" "Resistor_SMD:R_0805_2012Metric" (at 46.99 126.238 90)
       (effects (font (size 1.27 1.27)) hide)
     )
@@
       (effects (font (size 1.27 1.27)))
     )
-    (property "Footprint" "Resistor_SMD:R_0603_1608Metric" (at 100.33 94.488 90)
+    (property "Footprint" "Resistor_SMD:R_0805_2012Metric" (at 100.33 94.488 90)
       (effects (font (size 1.27 1.27)) hide)
     )
@@
       (effects (font (size 1.27 1.27)))
     )
-    (property "Footprint" "Resistor_SMD:R_0603_1608Metric" (at 121.92 162.052 90)
+    (property "Footprint" "Resistor_SMD:R_0805_2012Metric" (at 121.92 162.052 90)
       (effects (font (size 1.27 1.27)) hide)
     )
@@
       (effects (font (size 1.27 1.27)))
     )
-    (property "Footprint" "Resistor_SMD:R_0603_1608Metric" (at 100.33 85.598 90)
+    (property "Footprint" "Resistor_SMD:R_0805_2012Metric" (at 100.33 85.598 90)
       (effects (font (size 1.27 1.27)) hide)
     )
@@
       (effects (font (size 1.27 1.27)))
     )
-    (property "Footprint" "Resistor_SMD:R_0603_1608Metric" (at 249.428 81.28 90)
+    (property "Footprint" "Resistor_SMD:R_0805_2012Metric" (at 249.428 81.28 90)
       (effects (font (size 1.27 1.27)) hide)
     )
@@
       (effects (font (size 1.27 1.27)))
     )
-    (property "Footprint" "Resistor_SMD:R_0603_1608Metric" (at 161.29 159.258 90)
+    (property "Footprint" "Resistor_SMD:R_0805_2012Metric" (at 161.29 159.258 90)
       (effects (font (size 1.27 1.27)) hide)
     )
@@
       (effects (font (size 1.27 1.27)) (justify left))
     )
-    (property "Footprint" "Diode_SMD:D_0603_1608Metric" (at 110.49 80.01 0)
+    (property "Footprint" "Diode_SMD:D_0805_2012Metric" (at 110.49 80.01 0)
       (effects (font (size 1.27 1.27)) hide)
     )
@@
       (effects (font (size 1.27 1.27)))
     )
-    (property "Footprint" "Resistor_SMD:R_0603_1608Metric" (at 161.29 76.708 90)
+    (property "Footprint" "Resistor_SMD:R_0805_2012Metric" (at 161.29 76.708 90)
       (effects (font (size 1.27 1.27)) hide)
     )
@@
       (effects (font (size 1.27 1.27)))
     )
-    (property "Footprint" "Resistor_SMD:R_0603_1608Metric" (at 36.322 93.98 90)
+    (property "Footprint" "Resistor_SMD:R_0805_2012Metric" (at 36.322 93.98 90)
       (effects (font (size 1.27 1.27)) hide)
     )
@@
       (effects (font (size 1.27 1.27)))
     )
-    (property "Footprint" "Resistor_SMD:R_0603_1608Metric" (at 82.55 52.578 90)
+    (property "Footprint" "Resistor_SMD:R_0805_2012Metric" (at 82.55 52.578 90)
       (effects (font (size 1.27 1.27)) hide)
     )
@@
       (effects (font (size 1.27 1.27)))
     )
-    (property "Footprint" "Resistor_SMD:R_0603_1608Metric" (at 31.75 50.038 90)
+    (property "Footprint" "Resistor_SMD:R_0805_2012Metric" (at 31.75 50.038 90)
       (effects (font (size 1.27 1.27)) hide)
     )
@@
       (effects (font (size 1.27 1.27)))
     )
-    (property "Footprint" "Resistor_SMD:R_0603_1608Metric" (at 31.75 55.118 90)
+    (property "Footprint" "Resistor_SMD:R_0805_2012Metric" (at 31.75 55.118 90)
       (effects (font (size 1.27 1.27)) hide)
     )
@@
       (effects (font (size 1.27 1.27)))
     )
-    (property "Footprint" "Resistor_SMD:R_0603_1608Metric" (at 85.09 132.588 90)
+    (property "Footprint" "Resistor_SMD:R_0805_2012Metric" (at 85.09 132.588 90)
       (effects (font (size 1.27 1.27)) hide)
     )
@@
       (effects (font (size 1.27 1.27)) (justify left))
     )
-    (property "Footprint" "Diode_SMD:D_0603_1608Metric" (at 113.03 160.02 0)
+    (property "Footprint" "Diode_SMD:D_0805_2012Metric" (at 113.03 160.02 0)
       (effects (font (size 1.27 1.27)) hide)
     )
@@
       (effects (font (size 1.27 1.27)))
     )
-    (property "Footprint" "Resistor_SMD:R_0603_1608Metric" (at 102.87 165.608 90)
+    (property "Footprint" "Resistor_SMD:R_0805_2012Metric" (at 102.87 165.608 90)
       (effects (font (size 1.27 1.27)) hide)
     )
@@
       (effects (font (size 1.27 1.27)))
     )
-    (property "Footprint" "Resistor_SMD:R_0603_1608Metric" (at 288.798 102.87 90)
+    (property "Footprint" "Resistor_SMD:R_0805_2012Metric" (at 288.798 102.87 90)
       (effects (font (size 1.27 1.27)) hide)
     )
@@
       (effects (font (size 1.27 1.27)))
     )
-    (property "Footprint" "Resistor_SMD:R_0603_1608Metric" (at 190.5 89.408 90)
+    (property "Footprint" "Resistor_SMD:R_0805_2012Metric" (at 190.5 89.408 90)
       (effects (font (size 1.27 1.27)) hide)
     )
@@
       (effects (font (size 1.27 1.27)))
     )
-    (property "Footprint" "Resistor_SMD:R_0603_1608Metric" (at 36.322 40.64 90)
+    (property "Footprint" "Resistor_SMD:R_0805_2012Metric" (at 36.322 40.64 90)
       (effects (font (size 1.27 1.27)) hide)
     )
@@
       (effects (font (size 1.27 1.27)))
     )
-    (property "Footprint" "Resistor_SMD:R_0603_1608Metric" (at 31.75 108.458 90)
+    (property "Footprint" "Resistor_SMD:R_0805_2012Metric" (at 31.75 108.458 90)
       (effects (font (size 1.27 1.27)) hide)
     )
@@
       (effects (font (size 1.27 1.27)))
     )
-    (property "Footprint" "Diode_SMD:D_0603_1608Metric" (at 280.67 95.25 0)
+    (property "Footprint" "Diode_SMD:D_0805_2012Metric" (at 280.67 95.25 0)
       (effects (font (size 1.27 1.27)) hide)
     )
@@
       (effects (font (size 1.27 1.27)))
     )
-    (property "Footprint" "Resistor_SMD:R_0603_1608Metric" (at 31.75 103.378 90)
+    (property "Footprint" "Resistor_SMD:R_0805_2012Metric" (at 31.75 103.378 90)
       (effects (font (size 1.27 1.27)) hide)
     )
@@
       (effects (font (size 1.27 1.27)))
     )
-    (property "Footprint" "Diode_SMD:D_0603_1608Metric" (at 101.6 152.4 0)
+    (property "Footprint" "Diode_SMD:D_0805_2012Metric" (at 101.6 152.4 0)
       (effects (font (size 1.27 1.27)) hide)
     )
@@
       (effects (font (size 1.27 1.27)) (justify left))
     )
-    (property "Footprint" "Resistor_SMD:R_0603_1608Metric" (at 202.692 115.57 90)
+    (property "Footprint" "Resistor_SMD:R_0805_2012Metric" (at 202.692 115.57 90)
       (effects (font (size 1.27 1.27)) hide)
     )
@@
       (effects (font (size 1.27 1.27)))
     )
-    (property "Footprint" "Resistor_SMD:R_0603_1608Metric" (at 249.428 69.85 90)
+    (property "Footprint" "Resistor_SMD:R_0805_2012Metric" (at 249.428 69.85 90)
       (effects (font (size 1.27 1.27)) hide)
     )
@@
       (effects (font (size 1.27 1.27)))
     )
-    (property "Footprint" "Diode_SMD:D_0603_1608Metric" (at 99.06 72.39 0)
-      (effects (font (size 1.27 1.27)) hide)
-    )
+    (property "Footprint" "Diode_SMD:D_0805_2012Metric" (at 99.06 72.39 0)
+      (effects (font (size 1.27 1.27)) hide)
+    )
